Commit message: Update table.urdf

File: sawyer_gazebo_env/models/table/table.urdf (robot description, URDF)
Before this commit: robot table, 1 links, 0 joints
Links:
- added link world
Joints:
- added joint world_table: type fixed, parent world, child table, origin xyz=0.05 0.0 0.0 rpy=0 0 0, axis 1 0 0
