Commit message: Add Behavioral Cloning initial code

File: sawyer_gazebo_env/models/camera/camera.urdf.xacro (robot description, xacro)
@@ -27,5 +27,6 @@
     <parent link="world" />
     <child link = "camera" />
-    <origin xyz="0.7 0.0 1.4" rpy="0.0 1.57 0.0" />
+    <!-- <origin xyz="0.7 0.0 1.4" rpy="0.0 1.57 0.0" /> -->
+    <origin xyz="0.7 0.0 1.6" rpy="0.0 1.57 0.0" />
   </joint>
   <gazebo reference="camera">
@@ -61,3 +62,117 @@
   </sensor>
  </gazebo>
+   <link name="camera2">
+  <collision>
+    <origin xyz="0 0 0" rpy="0 0 0"/>
+    <geometry>
+      <box size="${cameraSize} ${cameraSize} ${cameraSize}"/>
+    </geometry>
+  </collision>
+  <visual>
+    <origin xyz="0 0 0" rpy="0 0 0"/>
+    <geometry>
+      <box size="${cameraSize} ${cameraSize} ${cameraSize}"/>
+    </geometry>
+    <material name="blue"/>
+  </visual>
+  <inertial>
+        <mass value="0.001" />
+        <origin xyz="0 0 0" rpy="0 0 0" />
+        <inertia ixx="0.0001" ixy="0" ixz="0" iyy="0.0001" iyz="0" izz="0.0001" />
+      </inertial>
+</link>
+<joint name="camera_joint2" type="fixed">
+    <parent link="world" />
+    <child link = "camera2" />
+    <origin xyz="0.7 1 1" rpy="0 0 -1.57" />
+  </joint>
+  <gazebo reference="camera2">
+  <material>Gazebo/Blue</material>
+  <sensor type="camera" name="camera2">
+    <update_rate>30.0</update_rate>
+    <camera name="head2">
+      <horizontal_fov>1.3962634</horizontal_fov>
+      <image>
+        <width>800</width>
+        <height>800</height>
+        <format>R8G8B8</format>
+      </image>
+      <clip>
+        <near>0.02</near>
+        <far>300</far>
+      </clip>
+    </camera>
+    <plugin name="camera_controller2" filename="libgazebo_ros_camera.so">
+      <alwaysOn>true</alwaysOn>
+      <updateRate>0.0</updateRate>
+      <cameraName>right_camera/camera</cameraName>
+      <imageTopicName>image_raw</imageTopicName>
+      <cameraInfoTopicName>camera_info</cameraInfoTopicName>
+      <frameName>camera_link2</frameName>
+      <hackBaseline>0.07</hackBaseline>
+      <distortionK1>0.0</distortionK1>
+      <distortionK2>0.0</distortionK2>
+      <distortionK3>0.0</distortionK3>
+      <distortionT1>0.0</distortionT1>
+      <distortionT2>0.0</distortionT2>
+    </plugin>
+  </sensor>
+ </gazebo>
+ <link name="camera3">
+  <collision>
+    <origin xyz="0 0 0" rpy="0 0 0"/>
+    <geometry>
+      <box size="${cameraSize} ${cameraSize} ${cameraSize}"/>
+    </geometry>
+  </collision>
+  <visual>
+    <origin xyz="0 0 0" rpy="0 0 0"/>
+    <geometry>
+      <box size="${cameraSize} ${cameraSize} ${cameraSize}"/>
+    </geometry>
+    <material name="blue"/>
+  </visual>
+  <inertial>
+        <mass value="0.001" />
+        <origin xyz="0 0 0" rpy="0 0 0" />
+        <inertia ixx="0.0001" ixy="0" ixz="0" iyy="0.0001" iyz="0" izz="0.0001" />
+      </inertial>
+</link>
+<joint name="camera_joint3" type="fixed">
+    <parent link="world" />
+    <child link = "camera3" />
+    <origin xyz="2 0 1" rpy="0.0 0.0 -3.14" />
+  </joint>
+  <gazebo reference="camera3">
+  <material>Gazebo/Blue</material>
+  <sensor type="camera" name="camera3">
+    <update_rate>30.0</update_rate>
+    <camera name="head3">
+      <horizontal_fov>1.3962634</horizontal_fov>
+      <image>
+        <width>800</width>
+        <height>800</height>
+        <format>R8G8B8</format>
+      </image>
+      <clip>
+        <near>0.02</near>
+        <far>300</far>
+      </clip>
+    </camera>
+    <plugin name="camera_controller3" filename="libgazebo_ros_camera.so">
+      <alwaysOn>true</alwaysOn>
+      <updateRate>0.0</updateRate>
+      <cameraName>front_camera/camera</cameraName>
+      <imageTopicName>image_raw</imageTopicName>
+      <cameraInfoTopicName>camera_info</cameraInfoTopicName>
+      <frameName>camera_link3</frameName>
+      <hackBaseline>0.07</hackBaseline>
+      <distortionK1>0.0</distortionK1>
+      <distortionK2>0.0</distortionK2>
+      <distortionK3>0.0</distortionK3>
+      <distortionT1>0.0</distortionT1>
+      <distortionT2>0.0</distortionT2>
+    </plugin>
+  </sensor>
+ </gazebo>
 </robot>

File: sawyer_gazebo_env/models/plate/plate.urdf (robot description, URDF)
Before this commit: robot plate, 1 links, 0 joints
Links:
- link plate: geometry collision mesh filename=package://sawyer_gazebo_env/models/plate/plate.STL; visual mesh filename=package://sawyer_gazebo_env/models/plate/plate.STL

Commit message: Recording is back!

File: sawyer_gazebo_env/models/camera/camera.urdf.xacro (robot description, xacro)
@@ -27,6 +27,6 @@
     <parent link="world" />
     <child link = "camera" />
-    <!-- <origin xyz="0.7 0.0 1.4" rpy="0.0 1.57 0.0" /> -->
-    <origin xyz="0.7 0.0 1.6" rpy="0.0 1.57 0.0" />
+    <origin xyz="0.7 0.0 1.4" rpy="0.0 1.57 0.0" />
+    <!-- <origin xyz="0.7 0.0 1.6" rpy="0.0 1.57 0.0" /> -->
   </joint>
   <gazebo reference="camera">

File: sawyer_gazebo_env/models/table/table.urdf (robot description, URDF)
Before this commit: robot table, 2 links, 1 joints
Links:
- removed link world
Joints:
- removed joint world_table

Commit message: Firse minor update

File: sawyer_gazebo_env/models/camera/camera.urdf.xacro (robot description, xacro)
@@ -27,5 +27,5 @@
     <parent link="world" />
     <child link = "camera" />
-    <origin xyz="0.7 0.0 1.4" rpy="0.0 1.57 0.0" />
+    <origin xyz="0.62 0.0 1.4" rpy="0.0 1.57 0.0" />
     <!-- <origin xyz="0.7 0.0 1.6" rpy="0.0 1.57 0.0" /> -->
   </joint>

Commit message: So many changes, I forgot how many. Works.

File: sawyer_gazebo_env/models/camera/camera.urdf.xacro (robot description, xacro)
@@ -27,12 +27,173 @@
     <parent link="world" />
     <child link = "camera" />
+    <!-- <origin xyz="1.0 0.0 1.5" rpy="0.0 2.355398 0.0" /> -->
+    <!-- <origin xyz= "1.34918 -0.437414 1.024695" rpy="0 0.399643 2.75619" /> -->
+    <origin xyz="0.62 0.0 1.4" rpy="0.0 1.57 3.14" />
+    <!-- <origin xyz="0.62 0.0 1.4" rpy="0.0 1.57 0.0" /> -->
+    <!-- <origin xyz="0.7 0.0 1.6" rpy="0.0 1.57 0.0" /> -->
+   <!--  <origin xyz="1.12 0.5 1.4" rpy="0.0 1.57 3.14" /> -->
+  </joint>
+  <gazebo reference="camera">
+  <material>Gazebo/Grey</material>
+ <sensor type="camera" name="camera1">
+    <update_rate>30.0</update_rate>
+    <camera name="head">
+      <horizontal_fov>1.3962634</horizontal_fov>
+      <image>
+        <width>200</width>
+        <height>200</height>
+        <format>R8G8B8</format>
+      </image>
+      <clip>
+        <near>0.02</near>
+        <far>300</far>
+      </clip>
+    </camera>
+    <plugin name="camera_controller" filename="libgazebo_ros_camera.so">
+      <alwaysOn>true</alwaysOn>
+      <updateRate>0.0</updateRate>
+      <cameraName>top_camera/camera</cameraName>
+      <imageTopicName>image_raw</imageTopicName>
+      <cameraInfoTopicName>camera_info</cameraInfoTopicName>
+      <frameName>camera_link</frameName>
+      <hackBaseline>0.07</hackBaseline>
+      <distortionK1>0.0</distortionK1>
+      <distortionK2>0.0</distortionK2>
+      <distortionK3>0.0</distortionK3>
+      <distortionT1>0.0</distortionT1>
+      <distortionT2>0.0</distortionT2>
+    </plugin>
+  </sensor>
+ </gazebo>
+ <link name="camera3">
+  <collision>
+    <origin xyz="0 0 0" rpy="0 0 0"/>
+    <geometry>
+      <box size="${cameraSize} ${cameraSize} ${cameraSize}"/>
+    </geometry>
+  </collision>
+  <visual>
+    <origin xyz="0 0 0" rpy="0 0 0"/>
+    <geometry>
+      <box size="${cameraSize} ${cameraSize} ${cameraSize}"/>
+    </geometry>
+    <material name="blue"/>
+  </visual>
+  <inertial>
+        <mass value="0.001" />
+        <origin xyz="0 0 0" rpy="0 0 0" />
+        <inertia ixx="0.0001" ixy="0" ixz="0" iyy="0.0001" iyz="0" izz="0.0001" />
+      </inertial>
+</link>
+<joint name="camera_joint3" type="fixed">
+    <parent link="world" />
+    <child link = "camera3" />
     <origin xyz="0.62 0.0 1.4" rpy="0.0 1.57 0.0" />
-    <!-- <origin xyz="0.7 0.0 1.6" rpy="0.0 1.57 0.0" /> -->
-  </joint>
-  <gazebo reference="camera">
-  <material>Gazebo/Blue</material>
-  <sensor type="camera" name="camera1">
-    <update_rate>30.0</update_rate>
-    <camera name="head">
+  </joint>
+  <gazebo reference="camera3">
+  <material>Gazebo/Grey</material>
+  <sensor type="camera" name="camera3">
+    <update_rate>30.0</update_rate>
+    <camera name="head3">
+      <horizontal_fov>1.3962634</horizontal_fov>
+      <image>
+        <width>200</width>
+        <height>200</height>
+        <format>R8G8B8</format>
+      </image>
+      <clip>
+        <near>0.02</near>
+        <far>300</far>
+      </clip>
+    </camera>
+    <plugin name="camera_controller3" filename="libgazebo_ros_camera.so">
+      <alwaysOn>true</alwaysOn>
+      <updateRate>0.0</updateRate>
+      <cameraName>really_top_camera/camera</cameraName>
+      <imageTopicName>image_raw</imageTopicName>
+      <cameraInfoTopicName>camera_info</cameraInfoTopicName>
+      <frameName>camera_link3</frameName>
+      <hackBaseline>0.07</hackBaseline>
+      <distortionK1>0.0</distortionK1>
+      <distortionK2>0.0</distortionK2>
+      <distortionK3>0.0</distortionK3>
+      <distortionT1>0.0</distortionT1>
+      <distortionT2>0.0</distortionT2>
+    </plugin>
+  </sensor>
+ </gazebo>
+<!-- <gazebo reference="camera">
+    <sensor type="depth" name="openni_camera_camera">
+        <always_on>1</always_on>
+        <visualize>true</visualize>
+        <camera>
+            <horizontal_fov>1.3962634</horizontal_fov>
+            <image>
+                <width>200</width>
+                <height>200</height>
+                <format>R8G8B8</format>
+            </image>
+            <depth_camera>
+            </depth_camera>
+            <clip>
+                <near>0.01</near>
+                <far>100</far>
+            </clip>
+        </camera>
+        <plugin name="camera_controller" filename="libgazebo_ros_openni_kinect.so">
+            <alwaysOn>true</alwaysOn>
+                <updateRate>30.0</updateRate>
+                <cameraName>camera</cameraName>
+                <frameName>openni_camera_link</frameName>
+            <imageTopicName>rgb/image_raw</imageTopicName>
+            <depthImageTopicName>depth/image_raw</depthImageTopicName>
+            <pointCloudTopicName>depth/points</pointCloudTopicName>
+            <cameraInfoTopicName>rgb/camera_info</cameraInfoTopicName>
+            <depthImageCameraInfoTopicName>depth/camera_info</depthImageCameraInfoTopicName>
+            <pointCloudCutoff>0.4</pointCloudCutoff>
+                <hackBaseline>0.07</hackBaseline>
+                <distortionK1>0.0</distortionK1>
+                <distortionK2>0.0</distortionK2>
+                <distortionK3>0.0</distortionK3>
+                <distortionT1>0.0</distortionT1>
+                <distortionT2>0.0</distortionT2>
+            <CxPrime>0.0</CxPrime>
+            <Cx>0.0</Cx>
+            <Cy>0.0</Cy>
+            <focalLength>0.0</focalLength>
+            </plugin>
+    </sensor>
+</gazebo>
+ -->
+<!-- <link name="camera2">
+  <collision>
+    <origin xyz="0 0 0" rpy="0 0 0"/>
+    <geometry>
+      <box size="${cameraSize} ${cameraSize} ${cameraSize}"/>
+    </geometry>
+  </collision>
+  <visual>
+    <origin xyz="0 0 0" rpy="0 0 0"/>
+    <geometry>
+      <box size="${cameraSize} ${cameraSize} ${cameraSize}"/>
+    </geometry>
+    <material name="blue"/>
+  </visual>
+  <inertial>
+        <mass value="0.001" />
+        <origin xyz="0 0 0" rpy="0 0 0" />
+        <inertia ixx="0.0001" ixy="0" ixz="0" iyy="0.0001" iyz="0" izz="0.0001" />
+      </inertial>
+</link>
+<joint name="camera_joint2" type="fixed">
+    <parent link="world" />
+    <child link = "camera2" />
+    <origin xyz="0.7 1 1" rpy="0 0 -1.57" />
+  </joint>
+  <gazebo reference="camera2">
+  <material>Gazebo/Grey</material>
+  <sensor type="camera" name="camera2">
+    <update_rate>30.0</update_rate>
+    <camera name="head2">
       <horizontal_fov>1.3962634</horizontal_fov>
       <image>
@@ -46,21 +207,21 @@
       </clip>
     </camera>
-    <plugin name="camera_controller" filename="libgazebo_ros_camera.so">
-      <alwaysOn>true</alwaysOn>
-      <updateRate>0.0</updateRate>
-      <cameraName>top_camera/camera</cameraName>
-      <imageTopicName>image_raw</imageTopicName>
-      <cameraInfoTopicName>camera_info</cameraInfoTopicName>
-      <frameName>camera_link</frameName>
-      <hackBaseline>0.07</hackBaseline>
-      <distortionK1>0.0</distortionK1>
-      <distortionK2>0.0</distortionK2>
-      <distortionK3>0.0</distortionK3>
-      <distortionT1>0.0</distortionT1>
-      <distortionT2>0.0</distortionT2>
-    </plugin>
-  </sensor>
- </gazebo>
-   <link name="camera2">
+    <plugin name="camera_controller2" filename="libgazebo_ros_camera.so">
+      <alwaysOn>true</alwaysOn>
+      <updateRate>0.0</updateRate>
+      <cameraName>right_camera/camera</cameraName>
+      <imageTopicName>image_raw</imageTopicName>
+      <cameraInfoTopicName>camera_info</cameraInfoTopicName>
+      <frameName>camera_link2</frameName>
+      <hackBaseline>0.07</hackBaseline>
+      <distortionK1>0.0</distortionK1>
+      <distortionK2>0.0</distortionK2>
+      <distortionK3>0.0</distortionK3>
+      <distortionT1>0.0</distortionT1>
+      <distortionT2>0.0</distortionT2>
+    </plugin>
+  </sensor>
+ </gazebo>
+ <link name="camera3">
   <collision>
     <origin xyz="0 0 0" rpy="0 0 0"/>
@@ -82,14 +243,14 @@
       </inertial>
 </link>
-<joint name="camera_joint2" type="fixed">
-    <parent link="world" />
-    <child link = "camera2" />
-    <origin xyz="0.7 1 1" rpy="0 0 -1.57" />
-  </joint>
-  <gazebo reference="camera2">
-  <material>Gazebo/Blue</material>
-  <sensor type="camera" name="camera2">
-    <update_rate>30.0</update_rate>
-    <camera name="head2">
+<joint name="camera_joint3" type="fixed">
+    <parent link="world" />
+    <child link = "camera3" />
+    <origin xyz="2 0 1" rpy="0.0 0.0 -3.14" />
+  </joint>
+  <gazebo reference="camera3">
+  <material>Gazebo/Grey</material>
+  <sensor type="camera" name="camera3">
+    <update_rate>30.0</update_rate>
+    <camera name="head3">
       <horizontal_fov>1.3962634</horizontal_fov>
       <image>
@@ -103,61 +264,4 @@
       </clip>
     </camera>
-    <plugin name="camera_controller2" filename="libgazebo_ros_camera.so">
-      <alwaysOn>true</alwaysOn>
-      <updateRate>0.0</updateRate>
-      <cameraName>right_camera/camera</cameraName>
-      <imageTopicName>image_raw</imageTopicName>
-      <cameraInfoTopicName>camera_info</cameraInfoTopicName>
-      <frameName>camera_link2</frameName>
-      <hackBaseline>0.07</hackBaseline>
-      <distortionK1>0.0</distortionK1>
-      <distortionK2>0.0</distortionK2>
-      <distortionK3>0.0</distortionK3>
-      <distortionT1>0.0</distortionT1>
-      <distortionT2>0.0</distortionT2>
-    </plugin>
-  </sensor>
- </gazebo>
- <link name="camera3">
-  <collision>
-    <origin xyz="0 0 0" rpy="0 0 0"/>
-    <geometry>
-      <box size="${cameraSize} ${cameraSize} ${cameraSize}"/>
-    </geometry>
-  </collision>
-  <visual>
-    <origin xyz="0 0 0" rpy="0 0 0"/>
-    <geometry>
-      <box size="${cameraSize} ${cameraSize} ${cameraSize}"/>
-    </geometry>
-    <material name="blue"/>
-  </visual>
-  <inertial>
-        <mass value="0.001" />
-        <origin xyz="0 0 0" rpy="0 0 0" />
-        <inertia ixx="0.0001" ixy="0" ixz="0" iyy="0.0001" iyz="0" izz="0.0001" />
-      </inertial>
-</link>
-<joint name="camera_joint3" type="fixed">
-    <parent link="world" />
-    <child link = "camera3" />
-    <origin xyz="2 0 1" rpy="0.0 0.0 -3.14" />
-  </joint>
-  <gazebo reference="camera3">
-  <material>Gazebo/Blue</material>
-  <sensor type="camera" name="camera3">
-    <update_rate>30.0</update_rate>
-    <camera name="head3">
-      <horizontal_fov>1.3962634</horizontal_fov>
-      <image>
-        <width>800</width>
-        <height>800</height>
-        <format>R8G8B8</format>
-      </image>
-      <clip>
-        <near>0.02</near>
-        <far>300</far>
-      </clip>
-    </camera>
     <plugin name="camera_controller3" filename="libgazebo_ros_camera.so">
       <alwaysOn>true</alwaysOn>
@@ -176,3 +280,4 @@
   </sensor>
  </gazebo>
+ -->
 </robot>

File: sawyer_gazebo_env/models/peg_ft_coarse/peg_ft.urdf (robot description, URDF)
Before this commit: robot peg_ft, 1 links, 0 joints
Links:
- link peg_ft: geometry collision mesh filename=package://sawyer_gazebo_env/models/peg_ft_coarse/high_res_c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; visual mesh filename=package://sawyer_gazebo_env/models/peg_ft_fine/peg_ft_fine.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

Commit message: Corrected peg-in-hole. Add peg, remove gripper.

File: sawyer_gazebo_env/models/camera/camera.urdf.xacro (robot description, xacro)
@@ -35,5 +35,5 @@
   </joint>
   <gazebo reference="camera">
-  <material>Gazebo/Grey</material>
+  <material>Gazebo/GreyTransparent</material>
  <sensor type="camera" name="camera1">
     <update_rate>30.0</update_rate>

File: sawyer_gazebo_env/models/semicircle/semicircle.urdf (robot description, URDF)
Before this commit: robot plate, 1 links, 0 joints
Links:
- removed link plate
- added link semicircle, mass 0.19635; collision mesh filename=package://sawyer_gazebo_env/models/semicircle/semicircle.STL; visual mesh filename=package://sawyer_gazebo_env/models/semicircle/semicircle.STL

File: sawyer_gazebo_env/models/sphere/sphere.urdf (robot description, URDF)
Before this commit: robot plate, 1 links, 0 joints
Links:
- removed link plate
- added link sphere, mass 0.39793; collision mesh filename=package://sawyer_gazebo_env/models/sphere/sphere.STL; visual mesh filename=package://sawyer_gazebo_env/models/sphere/sphere.STL

Commit message: Updated camera pos

File: sawyer_gazebo_env/models/camera/camera.urdf.xacro (robot description, xacro)
@@ -66,5 +66,5 @@
   </sensor>
  </gazebo>
- <link name="camera3">
+ <!-- <link name="camera3">
   <collision>
     <origin xyz="0 0 0" rpy="0 0 0"/>
@@ -123,4 +123,5 @@
   </sensor>
  </gazebo>
+ -->
 <!-- <gazebo reference="camera">
     <sensor type="depth" name="openni_camera_camera">
